File: Controller_T41_rev0.3.sch (KiCad schematic (older format))
At the start: 54 parts, among them J1 8P8C_x4, J2 8P8C_x4, J3 Screw_Terminal_01x02, J4 RJ45_LED, U1 Teensy4.1, U2 AMS1117-5.0, U3 74HCT245, U4 74HCT245, U5 74HCT245, U6 74HCT245

Commit message: Smaller resistors, larger fuse, additional labeling on silkscreen
Parts:
- added J5: 5v Conn, Connector_PinHeader_2.54mm:PinHeader_1x02_P2.54mm_Vertical, symbol Connector:Conn_01x02_Male
- F1: footprint Fuse:Fuse_0603_1608Metric_Pad1.05x0.95mm_HandSolder -> Fuse:Fuse_1206_3216Metric_Pad1.42x1.75mm_HandSolder
Connections:
- wire segments 115 -> 124
Other:
- moved on the sheet: C1, C2, D1, D2, F1, FB1, R1, U2

Commit message: Minor Placement Updates
Changed lines of the file:
@@
 L logo:LOGO #G1
 U 1 1 5FF38EC2
-P 850 690
-F 0 "#G1" H 850 637 60  0001 C CNN
-F 1 "LOGO" H 850 743 60  0001 C CNN
-F 2 "Controller_T41_rev0.2:logo" H 850 690 50  0001 C CNN
-F 3 "" H 850 690 50  0001 C CNN
-	1    850  690
+P 10130 7510
+F 0 "#G1" H 10130 7457 60  0001 C CNN
+F 1 "LOGO" H 10130 7563 60  0001 C CNN
+F 2 "Controller_T41_rev0.2:logo" H 10130 7510 50  0001 C CNN
+F 3 "" H 10130 7510 50  0001 C CNN
+	1    10130 7510
 	1    0    0    -1
 $EndComp
